File: door_alarm_hw/door_open_alarm.kicad_sch (KiCad schematic)
At the start: 62 parts, among them Q1 CJ2301 S1, Q2 BSS138PW,115, Q3 CJ2301 S1, SW1 TS-1088-AR02016, SW2 TS-1088-AR02016, SW3 SS-12D10L5, SW4 MET-200, U1 ESP32-S3-MINI-1, U2 AP2114HA-3.3TRG1

Commit message: ++commit
Parts:
- R11: value 15k 1% -> 5.1k 1%
Changed lines of the file:
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@@
       (effects (font (size 1.27 1.27)) (justify left))
     )
-    (property "Value" "15k 1%" (at 116.84 173.99 0)
+    (property "Value" "5.1k 1%" (at 116.84 173.99 0)
       (effects (font (size 1.27 1.27)) (justify left))
     )
