File: door_alarm_hw/door_open_alarm.kicad_sch (KiCad schematic)
At the start: 62 parts, among them Q1 CJ2301 S1, Q2 BSS138PW,115, Q3 CJ2301 S1, SW1 TS-1088-AR02016, SW2 TS-1088-AR02016, SW3 SS-12D10L5, SW4 MET-200, U1 ESP32-S3-MINI-1, U2 AP2114HA-3.3TRG1

Commit message: Bulk change after component lib change
Parts:
- removed USB1: TYPE-C 16PIN 2MD(073), my_lib:USB-C-SMD_TYPE-C-6PIN-2MD-073, symbol my_symbol_library:TYPE-C16PIN2MD(073)
- added USB1: TYPE-C 16PIN 2MD(073), pepy_sym_lib:[USB_C_16P_RA_FEMALE]SHOU HAN TYPE-C 16PIN 2MD(073), symbol pepy_sym_lib:[USB_C_16P_RA_FEMALE]SHOU HAN TYPE-C 16PIN 2MD(073)
- C1: footprint Capacitor_SMD:C_0805_2012Metric -> pepy_sym_lib:[CAP_SMD]0805_2012Metric; symbol Device:C_Small -> pepy_sym_lib:[CAP_SMD]0805_2012Metric; LCSC Part (none) -> C49678
- C2, C3, C4, C5, C6, C7, C8: footprint Capacitor_SMD:C_0805_2012Metric -> pepy_sym_lib:[CAP_SMD]0805_2012Metric; symbol Device:C -> pepy_sym_lib:[CAP_SMD]0805_2012Metric; LCSC Part (none) -> C49678
- D1: footprint my_lib:SOT-666-6_L1.6-W1.2-P0.50-LS1.6-BR -> pepy_sym_lib:[ESD_PROT]STMicroelectronics USBLC6-2P6; symbol my_symbol_library:USBLC6-2P6 -> pepy_sym_lib:[ESD_PROT]STMicroelectronics USBLC6-2P6
- D2: renamed from LED1; footprint my_lib:[LED]Lite-On LTST-C190KRKT -> pepy_sym_lib:[LED]Lite-On LTST-C190KRKT; symbol my_symbol_library:LTST-C190KRKT -> pepy_sym_lib:[LED]Lite-On LTST-C190KRKT
- D3: renamed from LED2; footprint my_lib:[LED]Lite-On LTST-C190KRKT -> pepy_sym_lib:[LED]Lite-On LTST-C190KRKT; symbol my_symbol_library:LTST-C190KRKT -> pepy_sym_lib:[LED]Lite-On LTST-C190KRKT
- D4: renamed from D3; footprint my_lib:SOD-123_L2.8-W1.8-LS3.7-RD -> pepy_sym_lib:[SCHOTTKY_DIODE_40V]STMicroelectronics STPS140Z; symbol my_symbol_library:STPS140Z -> pepy_sym_lib:[SCHOTTKY_DIODE_40V]STMicroelectronics STPS140Z
- D5: renamed from D4; footprint my_lib:SOD-123_L2.8-W1.8-LS3.7-RD -> pepy_sym_lib:[SCHOTTKY_DIODE_40V]STMicroelectronics STPS140Z; symbol my_symbol_library:STPS140Z -> pepy_sym_lib:[SCHOTTKY_DIODE_40V]STMicroelectronics STPS140Z
- D6: renamed from D2; footprint my_lib:SOD-123_L2.8-W1.8-LS3.7-RD -> pepy_sym_lib:[SCHOTTKY_DIODE_40V]STMicroelectronics STPS140Z; symbol my_symbol_library:STPS140Z -> pepy_sym_lib:[SCHOTTKY_DIODE_40V]STMicroelectronics STPS140Z
- FID1, FID2, FID3: footprint Fiducial:Fiducial_0.5mm_Mask1mm -> (none); now left out of the parts list
- H1: footprint my_lib:[6P_HEADER_STR]XFCN PZ254V-11-06P -> pepy_sym_lib:[6P_HEADER_STR]XFCN PZ254V-11-06P; symbol my_symbol_library:PZ254V-11-06P -> pepy_sym_lib:[6P_HEADER_STR]XFCN PZ254V-11-06P
- H2, H3, H4: footprint MountingHole:MountingHole_2.2mm_M2_DIN965_Pad -> (none); now left out of the parts list
- L1: footprint my_lib:FILTER-SMD_4P-L2.0-W1.2-BL_DLW21H -> pepy_sym_lib:[COMMON_MODE_FILTER]Murata Electronics DLW21SN900SQ2L; symbol my_symbol_library:DLW21SN900SQ2L -> pepy_sym_lib:[COMMON_MODE_FILTER]Murata Electronics DLW21SN900SQ2L
- Q1, Q3: footprint my_lib:[PMOS]Jiangsu Changjing Electronics Technology Co., Ltd. CJ2301 S1 -> pepy_sym_lib:[PMOS]Jiangsu Changjing Electronics Technology Co., Ltd. CJ2301 S1; symbol my_symbol_library:CJ2301S1 -> pepy_sym_lib:[PMOS]Jiangsu Changjing Electronics Technology Co., Ltd. CJ2301 S1
- Q2: footprint my_lib:[NMOS]Nexperia BSS138PW,115 -> pepy_sym_lib:[NMOS]Nexperia BSS138PW,115; symbol my_symbol_library:BSS138PW,115 -> pepy_sym_lib:[NMOS]Nexperia BSS138PW,115
- R1, R10, R11, R12, R13, R14, R16, R17, R3, R5, R8, R9: footprint Resistor_SMD:R_0805_2012Metric -> pepy_sym_lib:[RES_SMD]0805_2012Metric; symbol Device:R_Small -> pepy_sym_lib:[RES_SMD]0805_2012Metric; LCSC Part (none) -> C17414
- R15, R2, R4, R6, R7: footprint Resistor_SMD:R_0805_2012Metric -> pepy_sym_lib:[RES_SMD]0805_2012Metric; symbol Device:R -> pepy_sym_lib:[RES_SMD]0805_2012Metric; LCSC Part (none) -> C17414
- REED_G1, REED_OUT1, TP10, TP9: footprint TestPoint:TestPoint_Pad_2.0x2.0mm -> (none)
- SW1, SW2: footprint my_lib:[TACTILE_SWITCH]XUNPU TS-1088-AR02016 -> pepy_sym_lib:[TACTILE_SWITCH]XUNPU TS-1088-AR02016; symbol my_symbol_library:TS-1088-AR02016 -> pepy_sym_lib:[TACTILE_SWITCH]XUNPU TS-1088-AR02016
- SW3: footprint my_lib:[SLIDE_SWITCH]XKB Connection SS-12D10L5 -> pepy_sym_lib:[SLIDE_SWITCH]XKB Connection SS-12D10L5; symbol my_symbol_library:SS-12D10L5 -> pepy_sym_lib:[SLIDE_SWITCH]XKB Connection SS-12D10L5
- SW4: now in the parts list
- TP1, TP11, TP2, TP3, TP4, TP5, TP6, TP7, TP8: footprint TestPoint:TestPoint_Pad_D1.0mm -> (none)
- U1: footprint PCM_Espressif:ESP32-S3-MINI-1 -> pepy_sym_lib:[MCU]Espressif Systems ESP32-S3-MINI-1-N8; symbol PCM_Espressif:ESP32-S3-MINI-1 -> pepy_sym_lib:[MCU]Espressif Systems ESP32-S3-MINI-1-N8
- U2: footprint my_lib:[LDO]Diodes Incorporated AP2114HA-3.3TRG1 -> pepy_sym_lib:[LDO]Diodes Incorporated AP2114HA-3.3TRG1; symbol my_symbol_library:AP2114HA-3.3TRG1 -> pepy_sym_lib:[LDO]Diodes Incorporated AP2114HA-3.3TRG1
Connections:
- net +3.3V: now also C2.2, C3.2, R13.2, R15.2, R6.2, R7.2; no longer C2.1, C3.1, R13.1, R15.1, R6.1, R7.1
- net BOOT0: now also C7.2, R7.1; no longer C7.1, R7.2
- net D+: now also USB1.6 (DP1), USB1.8 (DP2)
- net D-: now also USB1.5 (DN2), USB1.7 (DN1)
- net EN: now also R8.2; no longer R8.1
- net ESP_RESET: now also C6.2, R6.1; no longer C6.1, R6.2
- net GND: now also C1.1, C2.1, C3.1, C4.1, C6.1, C7.1, C8.1, R11.1, R14.1, R16.1, R17.1, R2.2, R4.2, R5.1, USB1.1 (GND), USB1.12 (GND); no longer C1.2, C2.2, C3.2, C4.2, C6.2, C7.2, C8.2, R11.2, R14.2, R16.2, R17.2, R2.1, R4.1, R5.2
- net LED_EN: now also R3.2; no longer R3.1
- net MEAS_EN: now also R10.2; no longer R10.1
- net SHIELD: now also C1.2, R5.2, USB1.13 (SHELL), USB1.14 (SHELL); no longer C1.1, R5.1
- net STRAP_3: now also R13.1, R16.2; no longer R13.2, R16.1
- net STRAP_45: now also R14.2; no longer R14.1
- net STRAP_46: now also R17.2; no longer R17.1
- net VBUS: now also R1.2, USB1.11 (VBUS), USB1.2 (VBUS); no longer R1.1
- net V_INPUT: now also C4.2, R8.1; no longer C4.1, R8.2
- net V_SENSE: now also C8.2, R11.2, R9.1; no longer C8.1, R11.1, R9.2
- net at Q3.2 (S): now also R15.1; no longer R15.2
- net at Q1.3 (D): now also R9.2; no longer R9.1
- net at D2.2 (A): now also R1.1; no longer R1.2
- net at D3.2 (A): now also R3.1; no longer R3.2
- net at Q2.1 (G), R12.1: now also R10.1; no longer R10.2
- new net: R4.1, USB1.10 (CC2)
- new net: R2.1, USB1.4 (CC1)
Other:
- moved on the sheet: D2, D5, R1, R10, R11, R12, R13, R14, R15, R16, R17, R2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

Commit message: Updating components and design as well as yaml
Parts:
- added TP?: TestPoint, pepy_sym_lib:[TEST_POINT]TestPoint_Pad_D1.0mm, symbol pepy_sym_lib:[TEST_POINT]TestPoint
- FID1, FID2, FID3: value Fiducial -> ~
- REED_G1: value REED_G -> GND
- SW4, TP3: now left out of the parts list
Connections:
- net +3.3V: now also C2.1, C3.1, R13.1, R15.1, R6.1, R7.1; no longer C2.2, C3.2, R13.2, R15.2, R6.2, R7.2
- net BOOT0: now also C7.1, R7.2; no longer C7.2, R7.1
- net EN: now also R8.1; no longer R8.2
- net ESP_RESET: now also C6.1, R6.2; no longer C6.2, R6.1
- net GND: now also C1.2, C2.2, C3.2, C4.2, C6.2, C7.2, C8.2, R11.2, R12.1, R14.2, R16.2, R17.2, R2.1, R4.1, R5.2; no longer C1.1, C2.1, C3.1, C4.1, C6.1, C7.1, C8.1, R11.1, R12.2, R14.1, R16.1, R17.1, R2.2, R4.2, R5.1
- net LED_EN: now also R3.1; no longer R3.2
- net MEAS_EN: now also R10.1; no longer R10.2
- net SHIELD: now also C1.1, R5.1; no longer C1.2, R5.2
- net STRAP_3: now also R13.2, R16.1; no longer R13.1, R16.2
- net STRAP_45: now also R14.1; no longer R14.2
- net STRAP_46: now also R17.1; no longer R17.2
- net VBUS: now also R1.1; no longer R1.2
- net V_INPUT: now also C4.1, R8.2; no longer C4.2, R8.1
- net V_SENSE: now also C8.1, R11.1, R9.2, TP?.1; no longer C8.2, R11.2, R9.1
- net at Q3.2 (S): now also R15.2; no longer R15.1
- net at Q1.3 (D): now also R9.1; no longer R9.2
- net at D2.2 (A): now also R1.2; no longer R1.1
- net at D3.2 (A): now also R3.2; no longer R3.1
- net at USB1.10 (CC2): now also R4.2; no longer R4.1
- net at USB1.4 (CC1): now also R2.2; no longer R2.1
- new net: Q2.1 (G), R10.2, R12.2
Other:
- moved on the sheet: C1, C2, C3, C4, C6, C7, C8

Commit message: Overhaul
Parts:
- removed D1: USBLC6-2P6, pepy_sym_lib:[ESD_PROT]STMicroelectronics USBLC6-2P6, symbol pepy_sym_lib:[ESD_PROT]STMicroelectronics USBLC6-2P6
- removed TP?: TestPoint, pepy_sym_lib:[TEST_POINT]TestPoint_Pad_D1.0mm, symbol pepy_sym_lib:[TEST_POINT]TestPoint
- added D1: IP4283CZ10-TBR,115, pepy_sym_lib:[ESD_PROT]Nexperia IP4283CZ10-TBR,115, symbol pepy_sym_lib:[ESD_PROT]Nexperia IP4283CZ10-TBR,115
- TP1, TP11, TP2, TP3, TP4, TP5, TP6, TP7, TP8: footprint (none) -> pepy_sym_lib:[TEST_POINT]TestPoint_Pad_D1.0mm
- TP10, TP9: footprint (none) -> pepy_sym_lib:[TEST_POINT]TestPoint_Pad_2.0x2.0mm
Connections:
- net USB_D+_FIL is gone; now on net USB_D+: L1.3, U1.24 (GPIO20/U1CTS/ADC2_CH9/CLK_OUT1/USB_D+)
- net USB_D-_FIL is gone; now on net USB_D-: L1.2, U1.23 (GPIO19/U1RTS/ADC2_CH8/CLK_OUT2/USB_D-)
- net D+: now also L1.4, D1.4 (TMDS_CH2-)
- net D-: now also L1.1, D1.2 (TMDS_CH1+)
- net GND: now also D1.3 (GND), D1.8 (GND)
- net USB_D+: no longer L1.4
- net USB_D-: no longer L1.1
- no-connect marks 27 -> 31
Other:
- moved on the sheet: L1

Commit message: change++
Connections:
- net D+: now also D1.7 (NC)
- net D-: now also D1.9 (NC)
Changed lines of the file:
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@@
 	)
 	(label "D-"
-		(at 101.6 40.64 0)
+		(at 101.6 41.91 0)
 		(fields_autoplaced yes)
 		(effects
@@
 	)
 	(label "D+"
-		(at 101.6 43.18 0)
+		(at 101.6 44.45 0)
 		(fields_autoplaced yes)
 		(effects
